File: mod1base.kicad_pcb (KiCad board)
At the start: 2 copper layers, 100 x 100 mm, 170 parts, among them J1 SWD, J10 OUT, J11 FAN, J2 USB, J3 12V 300mA, J4 COM, J5 5034801000, J6 COM, J7 LCD, J8 5034801000, J9 IN, Q1 IRLML6402, SW1 SOFT2, SW10 STORE, SW2 STORE, SW3 SOFT1, SW4 PRESETS, SW5 SOFT2, SW6 SOFT3, SW7 ALL_LOAD, SW8 EVE-JBBF2020B, SW9 EVE-JBBF2020B, U1 LM1117DT-3.3, U2 ATSAMD20G18A-AU, U3 FT230XS, U4 74HCT245PW, U5 AP3211

Commit message: Rewrite references
Parts:
- removed the R10 at (58.5, 27.5)
- added R27: 100, IPC7351-Nominal:RESC1608X50, F.Cu at (58.5, 27.5)
- renumbered C4 to C1, C11 to C10, C20 to C11, C19 to C12, C12 to C13, C18 to C14, C13 to C15, C15 to C16, C16 to C17, C17 to C18, C14 to C19, C5 to C2, C9 to C20, C23 to C21, C24 to C23, C10 to C24, C21 to C3, C3 to C4, C6 to C5, C1 to C6, C2 to C7, C7 to C9, DZ2 to DZ1, DZ1 to DZ2, J4 to J1, J3 to J10, J1 to J2, J10 to J3, J9 to J4, J7 to J5, J5 to J6, J8 to J7, J6 to J8, J2 to J9, MP4 to MP1, MP2 to MP10, MP3 to MP11, MP5 to MP2, MP6 to MP3, MP7 to MP4, MP8 to MP5, MP9 to MP6, MP10 to MP7, MP11 to MP8, MP1 to MP9, R18 to R10, R22 to R11, R31 to R12, R19 to R13, R32 to R14, R35 to R15, R20 to R16, R27 to R17, R33 to R18, R15 to R19, R14 to R2, R25 to R20, R28 to R21, R5 to R22, R36 to R23, R16 to R24, R4 to R25, R29 to R26, R11 to R28, R38 to R29, R13 to R3, R37 to R30, R8 to R31, R9 to R32, R12 to R33, R2 to R34, R6 to R35, R7 to R36, R24 to R37, R39 to R38, R30 to R4, R34 to R5, R17 to R6, R21 to R7, R23 to R8, R26 to R9, SW3 to SW1, SW9 to SW10, SW4 to SW2, SW5 to SW3, SW1 to SW4, SW6 to SW5, SW7 to SW6, SW2 to SW7, SW10 to SW8, SW8 to SW9, U2 to U1, U1 to U2, U4 to U3, U3 to U4
Connections:
- J6 pad 2: /SW0 -> /SW1
- J6 pad 3: /SW1 -> /SW2
- J6 pad 4: /SW2 -> /SW3
- J6 pad 5: /SW3 -> /SW4
- J6 pad 6: /SW4 -> /SW5
- J6 pad 7: /SW5 -> /SW6
- J7 pad 2: /SW0 -> /SW1
- J7 pad 3: /SW1 -> /SW2
- J7 pad 4: /SW2 -> /SW3
- J7 pad 5: /SW3 -> /SW4
- J7 pad 6: /SW4 -> /SW5
- J7 pad 7: /SW5 -> /SW6
- R19 pad 1: /SW0 -> /SW1
- R20 pad 1: /SW2 -> /SW3
- R21 pad 1: /SW4 -> /SW5
- R23 pad 1: /SW6 -> /SW8
- R24 pad 1: /SW1 -> /SW2
- R25 pad 1: /SW3 -> /SW4
- R26 pad 1: /SW5 -> /SW6
- SW1 pad 3: /SW0 -> /SW1
- SW2 pad 1: /SW1 -> /SW2
- SW3 pad 3: /SW2 -> /SW3
- SW4 pad 1: /SW3 -> /SW4
- SW5 pad 3: /SW4 -> /SW5
- SW6 pad 1: /SW5 -> /SW6
- SW8 pad 1: /SW6 -> /SW8
- U1 pad 1: /SW6 -> /SW8
- U1 pad 14: /SW0 -> /SW1
- U1 pad 15: /SW1 -> /SW2
- U1 pad 16: /SW2 -> /SW3
- U1 pad 19: /SW3 -> /SW4
- U1 pad 20: /SW4 -> /SW5
- U1 pad 21: /SW5 -> /SW6
Routing:
- net /SW6: track 6.40 -> 227.5 mm, vias 0 -> 2
- net /SW0: track 154.4 -> 0.00 mm
- net /SW2: track 185.7 -> 167.3 mm
- net /SW5: track 227.5 -> 212.8 mm
- net /SW4: track 212.8 -> 198.5 mm
- net /SW1: track 167.3 -> 154.4 mm, vias 2 -> 0
- net /SW3: track 198.5 -> 185.7 mm
- net /SW8: track 0.00 -> 6.40 mm

Commit message: More finalization
Parts:
- removed the REF** at (29.0, 59.0)
- removed the REF** at (32.5, 62.5)
- added J12: PWRSENSE, conn-100mil:CONN-100MIL-M-1x2, B.Cu at (35.0, 58.0)
- added R39: 4k7, IPC7351-Nominal:RESC1608X50, B.Cu at (40.2, 56.0)
- added R40: 4k7, IPC7351-Nominal:RESC1608X50, B.Cu at (38.5, 56.0)
Connections:
- U1 pad 34: Net-(U1-Pad34) -> /PWRSENSE
Routing:
- net /PWRSENSE: track 0.00 -> 17.2 mm
- net +3.3: track 534.8 -> 543.3 mm
- net Net-(J12-Pad1): track 0.00 -> 5.26 mm
- net /~RST: track 59.9 -> 63.5 mm
- net /SWCLK: track 47.5 -> 50.1 mm
- net /SWDIO: track 46.5 -> 48.4 mm

Commit message: More layout work
Parts:
- removed the REF** at (87.5, 62.5)
- removed the REF** at (72.5, 62.5)
- added REF**: VIA, VIA, F.Cu at (64.2, 70.0)
- added REF**: VIA, VIA, F.Cu at (62.5, 46.5)
- added REF**: VIA, VIA, F.Cu at (62.5, 12.5)
- added TP1: EXTRA, conn-test:TEST-SMD-SMALL, B.Cu at (36.8, 67.0)
- moved REF** 90.0 mm to (5.00, 5.00), turned to 90 degrees
- moved REF** 87.0 mm to (6.50, 93.5), turned to 90 degrees
- moved R34 85.3 mm to (4.00, 11.0), turned to 270 degrees
- moved C20 83.2 mm to (6.00, 11.0), turned to 270 degrees
- moved MP5 83.2 mm to (89.0, 94.0), turned to 90 degrees
- moved REF** 80.0 mm to (90.0, 10.0), turned to 90 degrees
- moved SW7 77.3 mm to (8.00, 85.0), turned to 180 degrees
- moved SW2 76.9 mm to (94.0, 82.0), turned to 90 degrees
- moved SW6 76.9 mm to (94.0, 18.0), turned to 90 degrees
- moved J9 76.4 mm to (16.0, 8.00), turned to 180 degrees
- moved MP9 76.1 mm to (6.00, 19.0), turned to 90 degrees
- moved R22 74.7 mm to (10.2, 84.8), turned to 270 degrees
- moved MP8 74.5 mm to (79.0, 6.00), turned to 90 degrees
- moved J6 73.5 mm to (5.00, 76.0), turned to 90 degrees
- moved C11 72.6 mm to (15.5, 88.0), turned to 180 degrees
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Routing:
- net +3.3: track 543.3 -> 489.9 mm, vias 6 -> 2
- net Net-(TP1-Pad1): track 0.00 -> 5.53 mm
- net /~RST: track 63.5 -> 58.6 mm
- net GND: track 119.5 -> 122.8 mm, vias 38 -> 39
- net Net-(J4-Pad2): track 12.7 -> 15.4 mm
- net /SWDIO: track 48.4 -> 45.8 mm
- net /SWCLK: track 50.1 -> 47.6 mm
- net /SW1: track 154.4 -> 155.9 mm
- net /SW2: track 167.3 -> 168.6 mm
- net /SW3: track 185.7 -> 187.0 mm
- net +5: track 223.9 -> 225.0 mm
- net /Rear breakaway/~CTS: track 27.4 -> 28.3 mm
- net /SW4: track 198.5 -> 199.4 mm
- net /SW5: track 212.8 -> 213.6 mm
- net /SW6: track 227.5 -> 228.3 mm
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Other:
- outline, holes or cut-outs redrawn
- board text added: "PSU CONTROLLER"
- board text added: "SEMIANALOG"
- board text removed: "MODULAR PSU CONTROLLER"

Commit message: More PCB revision (fab candidate)
Parts:
- removed the REF** at (5.00, 51.5)
- removed the REF** at (6.25, 51.5)
- removed the REF** at (7.50, 51.8)
- removed the REF** at (7.75, 52.8)
- removed the REF** at (5.00, 30.0)
- removed the REF** at (15.5, 42.5)
- added G***: LOGO, LOGO, F.Cu at (4.00, 96.0)
- added REF**111: VIA, VIA, F.Cu at (2.50, 32.5)
- added REF**112: VIA, VIA, F.Cu at (2.50, 33.5)
- added REF**113: VIA, VIA, F.Cu at (2.50, 34.5)
- added REF**121: VIA, VIA, F.Cu at (3.50, 33.0)
- added REF**122: VIA, VIA, F.Cu at (3.50, 34.0)
- added REF**123: VIA, VIA, F.Cu at (3.50, 35.0)
- added REF**131: VIA, VIA, F.Cu at (4.50, 32.5)
- added REF**1311: VIA, VIA, F.Cu at (7.50, 53.2)
- added REF**1312: VIA, VIA, F.Cu at (8.50, 53.2)
- added REF**1313: VIA, VIA, F.Cu at (9.50, 53.2)
- added REF**132: VIA, VIA, F.Cu at (4.50, 33.5)
- added REF**1321: VIA, VIA, F.Cu at (8.00, 52.2)
- added REF**1322: VIA, VIA, F.Cu at (9.00, 52.2)
- added REF**1323: VIA, VIA, F.Cu at (10.0, 52.2)
- added REF**133: VIA, VIA, F.Cu at (4.50, 34.5)
- added REF**1331: VIA, VIA, F.Cu at (7.50, 51.2)
- added REF**1332: VIA, VIA, F.Cu at (8.50, 51.2)
- added REF**1333: VIA, VIA, F.Cu at (9.50, 51.2)
- moved REF** 5.93 mm to (11.8, 90.8)
- moved L1 3.00 mm to (14.5, 48.5)
- moved Q1 3.00 mm to (15.0, 44.0)
- moved DZ2 2.50 mm to (8.00, 44.0)
- moved RT1 2.00 mm to (15.0, 39.5)
- moved C24 1.50 mm to (7.00, 39.0)
- moved J6 0.71 mm to (5.50, 76.5)
- moved U3 0.71 mm to (27.5, 81.5)
- moved R3 0.25 mm to (47.0, 85.5)
Routing:
- net GND: track 122.8 -> 152.3 mm, vias 39 -> 37
- net +12: track 19.6 -> 31.2 mm
- net /Rear breakaway/5VIN: track 13.7 -> 16.7 mm
- net +5: track 225.0 -> 222.4 mm
- net (no net): track 1.83 -> 0.00 mm, vias 1 -> 0
- net /SW4: track 199.4 -> 197.5 mm
- net /SW5: track 213.6 -> 211.8 mm
- net /SW6: track 228.3 -> 226.6 mm
- net /SW3: track 187.0 -> 185.2 mm
- net Net-(J10-Pad1): track 9.83 -> 8.56 mm
- net Net-(R8-Pad2): track 8.05 -> 7.12 mm
- net /SW2: track 168.6 -> 169.4 mm
- net /Panel/LCD_E: track 20.6 -> 19.9 mm
- net /Panel/LCD_D_~C: track 21.4 -> 20.7 mm
- net /Panel/LCD_D6: track 12.1 -> 12.8 mm
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
Commit message: Fab RC 2
Parts:
- added REF**: VIA, VIA, F.Cu at (47.0, 30.0)
- J10: value 12V 300mA -> 12V 500mA
- moved G*** 78.9 mm to (45.2, 28.8)
- moved REF** 1.00 mm to (44.5, 30.0)
Other:
- board text added: "MOD1BASE BUTTON EXTENSION"
- board text added: "MOD1BASE USB+POWER"
- board text removed: "MOD1BASE BUTTON EXTENSION REV A: 201511"
- board text removed: "MOD1BASE USB+POWER REV A: 201511"
- board text removed: "PSU CONTROLLER"
Changed lines of the file:
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@@
     (area -0.075001 -0.075001 100.075001 100.075001)
     (thickness 1.6)
-    (drawings 129)
+    (drawings 128)
     (tracks 1148)
     (zones 0)
-    (modules 186)
+    (modules 187)
     (nets 100)
   )
@@
     (add_net VBUS)
   )
+  (module VIA (layer F.Cu)
+    (at 47 30 90)
+    (fp_text reference REF** (at 0 0 90) (layer F.SilkS) hide
+      (effects (font (size 0.127 0.127) (thickness 0.03175)))
+    )
+    (fp_text value VIA (at 0 0 90) (layer F.Fab) hide
+      (effects (font (size 0.127 0.127) (thickness 0.03175)))
+    )
+    (pad 1 thru_hole circle (at 0 0 90) (size 0.8 0.8) (drill 0.4) (layers *.Cu)
+      (net 2 GND) (zone_connect 2))
+  )
   (module LOGO (layer F.Cu)
-    (at 4 96)
+    (at 45.25 28.75)
     (fp_text reference G*** (at 0 0) (layer F.SilkS) hide
       (effects (font (size 1.143 1.143) (thickness 0.1778)))
@@
       (effects (font (size 0.7 0.7) (thickness 0.15)))
     )
-    (fp_text value "12V 300mA" (at -18.5 23.25 270) (layer F.SilkS)
+    (fp_text value "12V 500mA" (at -18.5 23.25 270) (layer F.SilkS)
       (effects (font (size 1 1) (thickness 0.2)))
     )
@@
   )
   (module VIA (layer F.Cu)
-    (at 45.5 30 90)
+    (at 44.5 30 90)
     (fp_text reference REF** (at 0 0 90) (layer F.SilkS) hide
       (effects (font (size 0.127 0.127) (thickness 0.03175)))
@@
   (gr_line (start 1.5 67.5) (end 29 67.5) (layer Margin) (width 0.2))
   (gr_line (start 1.5 1.5) (end 1.5 67.5) (layer Margin) (width 0.2))
-  (gr_line (start 57.5 30.5) (end 57.5 31.5) (layer F.SilkS) (width 0.2))
-  (gr_line (start 57.5 31.5) (end 56.5 31.5) (layer F.SilkS) (width 0.2))
-  (gr_text SEMIANALOG (at 50 29.75) (layer F.SilkS)
+  (gr_line (start 57.5 30) (end 57.5 31) (layer F.SilkS) (width 0.2))
+  (gr_line (start 57.5 31) (end 56.5 31) (layer F.SilkS) (width 0.2))
+  (gr_text SEMIANALOG (at 52.25 28.25) (layer F.SilkS)
     (effects (font (size 0.7 0.7) (thickness 0.175)))
   )
-  (gr_text +3v3 (at 56 43.75 90) (layer F.SilkS)
+  (gr_text +3v3 (at 55 43.75 360) (layer F.SilkS)
     (effects (font (size 0.8 0.8) (thickness 0.2)))
   )
-  (gr_text G (at 56 38.5 90) (layer F.SilkS)
+  (gr_text G (at 56 38.5 360) (layer F.SilkS)
     (effects (font (size 0.8 0.8) (thickness 0.2)))
   )
-  (gr_text G (at 56 41 90) (layer F.SilkS)
+  (gr_text G (at 56 41 360) (layer F.SilkS)
     (effects (font (size 0.8 0.8) (thickness 0.2)))
   )
-  (gr_text ~RST (at 64 33.5 90) (layer F.SilkS)
+  (gr_text ~RST (at 64.5 33.5 360) (layer F.SilkS)
     (effects (font (size 0.8 0.8) (thickness 0.2)))
   )
-  (gr_text CLK (at 64 41 90) (layer F.SilkS)
+  (gr_text CLK (at 64.5 41 360) (layer F.SilkS)
     (effects (font (size 0.8 0.8) (thickness 0.2)))
   )
-  (gr_text IO (at 64 43.5 90) (layer F.SilkS)
+  (gr_text IO (at 64.5 43.5 360) (layer F.SilkS)
     (effects (font (size 0.8 0.8) (thickness 0.2)))
   )
-  (gr_text OUT (at 56.75 78.25 90) (layer F.SilkS)
+  (gr_text OUT (at 56.75 72 360) (layer F.SilkS)
     (effects (font (size 1 1) (thickness 0.25)))
   )
-  (gr_text G (at 54.25 77.75 90) (layer F.SilkS)
+  (gr_text G (at 54.25 72 360) (layer F.SilkS)
     (effects (font (size 1 1) (thickness 0.25)))
   )
-  (gr_text +3v3 (at 63.5 78 90) (layer F.SilkS)
+  (gr_text +3v3 (at 61.75 72 360) (layer F.SilkS)
     (effects (font (size 1 1) (thickness 0.25)))
   )
-  (gr_text +3v3 (at 62 95.75 90) (layer F.SilkS)
+  (gr_text +3v3 (at 63.5 89.25 360) (layer F.SilkS)
     (effects (font (size 1 1) (thickness 0.25)))
   )
-  (gr_text G (at 54.25 95 90) (layer F.SilkS)
+  (gr_text G (at 54.25 89.25 360) (layer F.SilkS)
     (effects (font (size 1 1) (thickness 0.25)))
   )
-  (gr_text IN (at 56.75 95 90) (layer F.SilkS)
+  (gr_text IN (at 56.75 89.25 360) (layer F.SilkS)
     (effects (font (size 1 1) (thickness 0.25)))
   )
@@
     (effects (font (size 1.5 1.5) (thickness 0.3)) (justify left))
   )
-  (gr_text "MOD1BASE BUTTON EXTENSION\nREV A: 201511" (at 98.25 91.25 270) (layer F.SilkS)
+  (gr_text "MOD1BASE\nBUTTON EXTENSION" (at 97.75 93.25 270) (layer F.SilkS)
     (effects (font (size 0.7 0.7) (thickness 0.125)))
   )
-  (gr_text "MOD1BASE USB+POWER\nREV A: 201511" (at 7.75 67) (layer F.SilkS)
+  (gr_text "MOD1BASE USB+POWER" (at 7.75 67) (layer F.SilkS)
     (effects (font (size 0.7 0.7) (thickness 0.175)))
   )
-  (gr_line (start 42 32) (end 42 24) (layer F.SilkS) (width 0.2))
-  (gr_line (start 58 32) (end 42 32) (layer F.SilkS) (width 0.2))
-  (gr_line (start 58 24) (end 58 32) (layer F.SilkS) (width 0.2))
-  (gr_line (start 42 24) (end 58 24) (layer F.SilkS) (width 0.2))
-  (gr_line (start 42.5 31.5) (end 43.5 31.5) (layer F.SilkS) (width 0.2))
-  (gr_line (start 42.5 30.5) (end 42.5 31.5) (layer F.SilkS) (width 0.2))
-  (gr_line (start 57.5 24.5) (end 57.5 25.5) (layer F.SilkS) (width 0.2))
-  (gr_line (start 56.5 24.5) (end 57.5 24.5) (layer F.SilkS) (width 0.2))
-  (gr_line (start 42.5 24.5) (end 42.5 25.5) (layer F.SilkS) (width 0.2))
-  (gr_line (start 43.5 24.5) (end 42.5 24.5) (layer F.SilkS) (width 0.2))
-  (gr_text "REV A: 201511" (at 50 31) (layer F.SilkS)
+  (gr_line (start 42 31.5) (end 42 23.5) (layer F.SilkS) (width 0.2))
+  (gr_line (start 58 31.5) (end 42 31.5) (layer F.SilkS) (width 0.2))
+  (gr_line (start 58 23.5) (end 58 31.5) (layer F.SilkS) (width 0.2))
+  (gr_line (start 42 23.5) (end 58 23.5) (layer F.SilkS) (width 0.2))
+  (gr_line (start 42.5 31) (end 43.5 31) (layer F.SilkS) (width 0.2))
+  (gr_line (start 42.5 30) (end 42.5 31) (layer F.SilkS) (width 0.2))
+  (gr_line (start 57.5 24) (end 57.5 25) (layer F.SilkS) (width 0.2))
+  (gr_line (start 56.5 24) (end 57.5 24) (layer F.SilkS) (width 0.2))
+  (gr_line (start 42.5 24) (end 42.5 25) (layer F.SilkS) (width 0.2))
+  (gr_line (start 43.5 24) (end 42.5 24) (layer F.SilkS) (width 0.2))
+  (gr_text "REV A: 201511" (at 52.25 29.75) (layer F.SilkS)
     (effects (font (size 0.7 0.7) (thickness 0.175)))
   )
-  (gr_text "PSU CONTROLLER" (at 50 28) (layer F.SilkS)
-    (effects (font (size 1.5 1) (thickness 0.25)))
-  )
-  (gr_text "MOD1BASE\n" (at 50 25.5) (layer F.SilkS)
+  (gr_text "MOD1BASE\n" (at 50 25) (layer F.SilkS)
     (effects (font (size 1.5 1.5) (thickness 0.375)))
   )

Commit message: Finalize revision A
Parts:
- moved TP1 1.25 mm to (38.0, 67.0)
Routing:
- net /Rear breakaway/~CTS: track 28.3 -> 30.6 mm
- net +5: track 222.4 -> 224.4 mm
- net /Rear breakaway/~RTS: track 50.2 -> 51.6 mm
