File: Panel.sch (KiCad schematic (older format))
At the start: 45 parts, among them J5 5034801000, J7 LCD, J8 5034801000, SW1 SOFT2, SW10 STORE, SW2 STORE, SW3 SOFT1, SW4 PRESETS, SW5 SOFT2, SW6 SOFT3, SW7 ALL_LOAD, SW8 EVE-JBBF2020B, SW9 EVE-JBBF2020B, U4 74HCT245PW

Commit message: Rewrite references
Parts:
- renumbered C11 to C10, C20 to C11, C19 to C12, C12 to C13, J7 to J5, J5 to J6, J8 to J7, MP8 to MP5, MP9 to MP6, MP10 to MP7, MP11 to MP8, R18 to R10, R22 to R11, R31 to R12, R19 to R13, R32 to R14, R35 to R15, R20 to R16, R27 to R17, R33 to R18, R15 to R19, R25 to R20, R28 to R21, R5 to R22, R36 to R23, R16 to R24, R4 to R25, R29 to R26, R30 to R4, R34 to R5, R17 to R6, R21 to R7, R23 to R8, R26 to R9, SW3 to SW1, SW9 to SW10, SW4 to SW2, SW5 to SW3, SW1 to SW4, SW6 to SW5, SW7 to SW6, SW2 to SW7, SW10 to SW8, SW8 to SW9, U4 to U3
Connections:
- net labels added: SW8, SW[1..8]
- net labels removed: SW0, SW[0..7]

Commit message: More finalization
Other:
- note added: "Layout note: grounded screw near interface connector"
- moved on the sheet: J6, J7, MP5, MP6, MP7, MP8

Commit message: Finalize revision A
Other:
- moved on the sheet: SW10A, SW9A
Changed lines of the file:
@@
 L ROTARY_PUSH SW9
 U 1 1 563C5431
-P 9250 1950
-F 0 "SW9" H 9535 2005 50  0000 L CNN
-F 1 "EVE-JBBF2020B" H 9535 1905 50  0000 L CNN
-F 2 "manuf:PANASONIC-EVEJB" H 9535 1855 60  0001 L CNN
-F 3 "" H 9250 2000 60  0000 C CNN
-F 4 "DIST DIGIKEY P12336-ND" H 9250 1950 60  0001 C CNN "BOM"
-	1    9250 1950
+P 9250 1850
+F 0 "SW9" H 9250 1500 50  0000 C CNN
+F 1 "EVE-JBBF2020B" H 9250 1350 50  0000 C CNN
+F 2 "manuf:PANASONIC-EVEJB" H 9535 1755 60  0001 L CNN
+F 3 "" H 9250 1900 60  0000 C CNN
+F 4 "DIST DIGIKEY P12336-ND" H 9250 1850 60  0001 C CNN "BOM"
+	1    9250 1850
 	1    0    0    -1
 $EndComp
@@
 L ROTARY_PUSH SW10
 U 1 1 563C5602
-P 9250 3550
-F 0 "SW10" H 9535 3605 50  0000 L CNN
-F 1 "EVE-JBBF2020B" H 9535 3505 50  0000 L CNN
-F 2 "manuf:PANASONIC-EVEJB" H 9250 3600 60  0001 C CNN
-F 3 "" H 9250 3600 60  0000 C CNN
-F 4 "DIST DIGIKEY P12336-ND" H 9250 3550 60  0001 C CNN "BOM"
-	1    9250 3550
+P 9250 3450
+F 0 "SW10" H 9250 3100 50  0000 C CNN
+F 1 "EVE-JBBF2020B" H 9250 2950 50  0000 C CNN
+F 2 "manuf:PANASONIC-EVEJB" H 9250 3500 60  0001 C CNN
+F 3 "" H 9250 3500 60  0000 C CNN
+F 4 "DIST DIGIKEY P12336-ND" H 9250 3450 60  0001 C CNN "BOM"
+	1    9250 3450
 	1    0    0    -1
 $EndComp
@@
 L GND #PWR029
 U 1 1 563C6398
-P 8800 3600
-F 0 "#PWR029" H 8800 3600 30  0001 C CNN
-F 1 "GND" H 8800 3530 30  0001 C CNN
-F 2 "" H 8800 3600 60  0000 C CNN
-F 3 "" H 8800 3600 60  0000 C CNN
-	1    8800 3600
+P 8800 3750
+F 0 "#PWR029" H 8800 3750 30  0001 C CNN
+F 1 "GND" H 8800 3680 30  0001 C CNN
+F 2 "" H 8800 3750 60  0000 C CNN
+F 3 "" H 8800 3750 60  0000 C CNN
+	1    8800 3750
 	1    0    0    -1
 $EndComp
@@
 L GND #PWR044
 U 1 1 563C8945
-P 8800 2000
-F 0 "#PWR044" H 8800 2000 30  0001 C CNN
-F 1 "GND" H 8800 1930 30  0001 C CNN
-F 2 "" H 8800 2000 60  0000 C CNN
-F 3 "" H 8800 2000 60  0000 C CNN
-	1    8800 2000
+P 8800 2150
+F 0 "#PWR044" H 8800 2150 30  0001 C CNN
+F 1 "GND" H 8800 2080 30  0001 C CNN
+F 2 "" H 8800 2150 60  0000 C CNN
+F 3 "" H 8800 2150 60  0000 C CNN
+	1    8800 2150
 	1    0    0    -1
 $EndComp
@@
 Text Label 8200 1750 0    50   ~ 0
 ROT0
-Text Label 8200 2150 0    50   ~ 0
+Text Label 8200 1950 0    50   ~ 0
 ROT1
 Text Label 8200 2650 0    50   ~ 0
@@
 Text Label 8200 3350 0    50   ~ 0
 ROT3
-Text Label 8200 3750 0    50   ~ 0
+Text Label 8200 3550 0    50   ~ 0
 ROT4
 Text Label 8200 4250 0    50   ~ 0
@@
 	8100 1650 8200 1750
 Entry Wire Line
-	8100 2050 8200 2150
+	8100 1850 8200 1950
 Entry Wire Line
 	8100 2550 8200 2650
@@
 	8100 3250 8200 3350
 Entry Wire Line
-	8100 3650 8200 3750
+	8100 3450 8200 3550
 Entry Wire Line
 	8100 4150 8200 4250
@@
 $EndComp
 Wire Wire Line
-	8800 3600 8800 3550
-Wire Wire Line
-	8800 3550 8900 3550
+	8800 3750 8800 3700
+Wire Wire Line
+	8800 3700 8900 3700
 Wire Wire Line
 	9650 2700 9650 2650
@@
 	8800 3350 8800 3250
 Wire Wire Line
-	8200 3750 8900 3750
-Wire Wire Line
-	8500 3750 8500 3250
+	8200 3550 8900 3550
 Wire Wire Line
 	8500 3950 8500 4000
@@
 	8500 2350 8500 2400
 Wire Wire Line
-	8800 2000 8800 1950
-Wire Wire Line
-	8800 1950 8900 1950
+	8800 2150 8800 2100
+Wire Wire Line
+	8800 2100 8900 2100
 Wire Wire Line
 	8200 1750 8900 1750
@@
 	8800 1750 8800 1650
 Wire Wire Line
-	8200 2150 8900 2150
-Wire Wire Line
-	8500 2150 8500 1650
+	8200 1950 8900 1950
 Wire Wire Line
 	8500 1400 8500 1450
@@
 	8800 3000 8800 3050
 Connection ~ 8800 1750
-Connection ~ 8500 2150
+Connection ~ 8500 1950
 Connection ~ 8500 2650
 Connection ~ 8800 3350
-Connection ~ 8500 3750
+Connection ~ 8500 3550
 Connection ~ 8500 4250
 Wire Wire Line
@@
 Text Notes 3200 7050 0    50   ~ 0
 Layout note: grounded screw near interface connector
+Wire Wire Line
+	8500 1650 8500 1950
+Wire Wire Line
+	8500 3550 8500 3250
 $EndSCHEMATC

Commit message: Update BOM references
Parts:
- SW1, SW2, SW3, SW4, SW5, SW6, SW7, SW8: BOM (none) -> DIST DIGIKEY EG1865-ND
- U3: BOM (none) -> DIST DIGIKEY 568-2809-5-ND
Changed lines of the file:
@@
 F 2 "manuf:ESWITCH-TL1105" H 4050 5000 60  0001 C CNN
 F 3 "" H 4050 5200 60  0000 C CNN
+F 4 "DIST DIGIKEY EG1865-ND" H 4050 5200 60  0001 C CNN "BOM"
 	1    4050 5200
 	1    0    0    -1
@@
 F 2 "manuf:ESWITCH-TL1105" H 5250 5000 60  0001 C CNN
 F 3 "" H 5250 5200 60  0000 C CNN
+F 4 "DIST DIGIKEY EG1865-ND" H 5250 5200 60  0001 C CNN "BOM"
 	1    5250 5200
 	1    0    0    -1
@@
 F 2 "manuf:ESWITCH-TL1105" H 6450 5000 60  0001 C CNN
 F 3 "" H 6450 5200 60  0000 C CNN
+F 4 "DIST DIGIKEY EG1865-ND" H 6450 5200 60  0001 C CNN "BOM"
 	1    6450 5200
 	1    0    0    -1
@@
 F 2 "manuf:ESWITCH-TL1105" H 6450 5800 60  0001 C CNN
 F 3 "" H 6450 6000 60  0000 C CNN
+F 4 "DIST DIGIKEY EG1865-ND" H 6450 6000 60  0001 C CNN "BOM"
 	1    6450 6000
 	1    0    0    -1
@@
 F 2 "manuf:ESWITCH-TL1105" H 9250 5000 60  0001 C CNN
 F 3 "" H 9250 5200 60  0000 C CNN
+F 4 "DIST DIGIKEY EG1865-ND" H 9250 5200 60  0001 C CNN "BOM"
 	1    9250 5200
 	1    0    0    -1
@@
 F 2 "manuf:ESWITCH-TL1105" H 4050 5800 60  0001 C CNN
 F 3 "" H 4050 6000 60  0000 C CNN
+F 4 "DIST DIGIKEY EG1865-ND" H 4050 6000 60  0001 C CNN "BOM"
 	1    4050 6000
 	1    0    0    -1
@@
 F 2 "manuf:ESWITCH-TL1105" H 5250 5800 60  0001 C CNN
 F 3 "" H 5250 6000 60  0000 C CNN
+F 4 "DIST DIGIKEY EG1865-ND" H 5250 6000 60  0001 C CNN "BOM"
 	1    5250 6000
 	1    0    0    -1
@@
 F 2 "manuf:ESWITCH-TL1105" H 7650 5000 60  0001 C CNN
 F 3 "" H 7650 5200 60  0000 C CNN
+F 4 "DIST DIGIKEY EG1865-ND" H 7650 5200 60  0001 C CNN "BOM"
 	1    7650 5200
 	1    0    0    -1
@@
 F 2 "IPC7351-Nominal:SOP65P640X110-20" H 4000 1900 50  0001 C CNN
 F 3 "" H 3950 2100 60  0000 C CNN
+F 4 "DIST DIGIKEY 568-2809-5-ND" H 4000 1900 60  0001 C CNN "BOM"
 	1    4000 1900
 	-1   0    0    -1
@@
 F 2 "IPC7351-Nominal:SOP65P640X110-20" H 1600 1150 50  0001 C CNN
 F 3 "" H 1550 1350 60  0000 C CNN
+F 4 "DIST DIGIKEY 568-2809-5-ND" H 1600 1150 60  0001 C CNN "BOM"
 	2    1600 1150
 	1    0    0    -1
