File: mod1base.sch (KiCad schematic (older format))
At the start: 22 parts, among them J1 SWD, J10 OUT, J4 COM, J9 IN, U1 LM1117DT-3.3, U2 ATSAMD20G18A-AU

Commit message: Rewrite references
Parts:
- renumbered C4 to C1, C5 to C2, C21 to C3, C3 to C4, C6 to C5, C1 to C6, C2 to C7, C7 to C9, J4 to J1, J1 to J2, J10 to J3, J9 to J4, MP4 to MP1, MP5 to MP2, MP6 to MP3, MP7 to MP4, R14 to R2, R13 to R3, U2 to U1, U1 to U2
Connections:
- net SW0 is gone; now on net SW1: U1.14 (PA09)
- net SW1: no longer U1.15 (PA10)
- net SW2: now also U1.15 (PA10); no longer U1.16 (PA11)
- net SW3: now also U1.16 (PA11); no longer U1.19 (PB10)
- net SW4: now also U1.19 (PB10); no longer U1.20 (PB11)
- net SW5: now also U1.20 (PB11); no longer U1.21 (PA12)
- net SW6: now also U1.21 (PA12); no longer U1.1 (PA00)
- new net SW8: U1.1 (PA00)

Commit message: More finalization
Parts:
- added J12: PWRSENSE, conn-100mil:CONN-100MIL-M-1x2, symbol CONN-100MIL-M-1x2
- added R39, R40: 4k7, IPC7351-Nominal:RESC1608X50, symbol R-0603
Connections:
- net +3.3: now also R40.1
- net GND: now also J12.2
- net PWRSENSE: now reaches U1.34 (PA25)
- net PWRSENSE: now also R39.2
- new net: J12.1, R39.1, R40.2
Other:
- note added: "Layout note: grounded screw near comm connectors"

Commit message: More layout work
Parts:
- added TP1: EXTRA, conn-test:TEST-SMD-SMALL, symbol TESTPOINT
Connections:
- net at U1.22 (PA13): now also TP1.1
Changed lines of the file:
@@
 	9000 3300 7800 3300
 Wire Bus Line
-	7800 3300 7700 3200
-Wire Bus Line
-	7700 3200 7700 1800
+	7700 3200 7800 3300
+Wire Bus Line
+	7700 1800 7700 3200
 Wire Bus Line
 	7800 3300 7700 3400
@@
 Wire Wire Line
 	7400 4500 9000 4500
+$Comp
+L TESTPOINT TP1
+U 1 1 564CEE37
+P 6400 3100
+F 0 "TP1" V 6400 3289 50  0000 L CNN
+F 1 "EXTRA" V 6450 3289 50  0001 L CNN
+F 2 "conn-test:TEST-SMD-SMALL" V 6450 3289 50  0001 L CNN
+F 3 "" H 6400 3100 50  0000 C CNN
+	1    6400 3100
+	0    1    1    0
+$EndComp
+Wire Wire Line
+	6400 3100 6200 3100
 $EndSCHEMATC

Commit message: Update BOM references
Parts:
- J2: BOM (none) -> DIST DIGIKEY ED1543-ND
- J3, J4: BOM (none) -> DIST DIGIKEY A19431-ND
- U1: BOM IC ATMEL ATSAMD20G18A-AU -> MCU ATMEL ATSAMD20G18A-AU
Connections:
- no-connect marks 7 -> 8
Other:
- note added: "Mating connector: A30980-ND"
Changed lines of the file:
@@
 F 2 "conn-100mil:CONN-100MIL-M-2x5" H 4075 3400 50  0001 C CNN
 F 3 "" H 4075 3400 50  0000 C CNN
+F 4 "DIST DIGIKEY ED1543-ND" H 4100 3400 60  0001 C CNN "BOM"
 	1    4100 3400
 	1    0    0    -1
@@
 F 2 "IPC7351-Nominal:QFP50P900X900X120-48" H 5650 1600 50  0001 C CNN
 F 3 "" H 5700 3300 50  0000 C CNN
-F 4 "IC ATMEL ATSAMD20G18A-AU" H 5600 5750 50  0001 C CNN "BOM"
+F 4 "MCU ATMEL ATSAMD20G18A-AU" H 5600 5750 50  0001 C CNN "BOM"
 	1    5600 3600
 	1    0    0    -1
@@
 F 2 "conn-100mil:CONN-100MIL-M-1x4-SHROUD" H 9550 5700 50  0001 C CNN
 F 3 "" H 9550 5700 50  0000 C CNN
+F 4 "DIST DIGIKEY A19431-ND" H 9550 5700 60  0001 C CNN "BOM"
 	1    9550 5700
 	1    0    0    -1
@@
 F 2 "conn-100mil:CONN-100MIL-M-1x4-SHROUD" H 9550 5200 50  0001 C CNN
 F 3 "" H 9550 5200 50  0000 C CNN
+F 4 "DIST DIGIKEY A19431-ND" H 9550 5200 60  0001 C CNN "BOM"
 	1    9550 5200
 	1    0    0    -1
@@
 	9000 3300 7800 3300
 Wire Bus Line
-	7700 3200 7800 3300
+	7800 3300 7700 3200
 Wire Bus Line
-	7700 1800 7700 3200
+	7700 3200 7700 1800
 Wire Bus Line
 	7800 3300 7700 3400
@@
 Wire Wire Line
 	6400 3100 6200 3100
+NoConn ~ 9500 5400
+Text Notes 8950 6300 0    50   ~ 0
+Mating connector: A30980-ND
 $EndSCHEMATC
